File: Hardware/0.4/0.4.kicad_sch (KiCad schematic)
At the start: 36 parts, among them J1 Acople Pull y LED, J1 Relay1, J2 Relay2, J3 Relay3, J4 Relay4, J5 Entrada 220, J6 Entrada 5V, K1 G5V-1, K2 G5V-1, K3 G5V-1, K4 G5V-1, Q1 S8050, Q2 S8050, Q3 S8050, Q4 S8050, SW2 SW_SPDT, U1 PC817, U2 PC817, U3 ESP32_DevKit_V1_DOIT, U4 PC817, U5 PC817, U6 Fuente Swiching 5V

Commit message: Subiendo imágenes esquemático master
Changed lines of the file:
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@@
     (in_bom yes) (on_board yes) (dnp no) (fields_autoplaced)
     (property "Reference" "J2" (at 269.24 58.42 0)
-      (effects (font (size 1.524 1.524)))
+      (effects (font (size 1.524 1.524)) hide)
     )
     (property "Value" "Relay2" (at 269.24 60.96 0)
